File: FMP3_PLAYER_CIRCUIT_ITER_2/FMP3_PLAYER.kicad_pcb (KiCad board)
At the start: 2 copper layers, 114 x 39.5 mm, 47 parts, among them J1 USB_C_Receptacle_PowerOnly_6P, J2 AudioJack3, J3 ISP, Q1 PMOS, Q2 PMOS, SW1 SW_L, SW2 SW_D, SW3 SW_R, SW4 SW_U, SW5 SW_SPDT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

Commit message: Second iteration complete, much cheaper to manufacture
Parts:
- moved C10 15.2 mm to (116.5, 43.5), turned to 90 degrees
- moved R9 13.0 mm to (113.5, 46.5), turned to 180 degrees
- moved R8 9.62 mm to (119.0, 46.5), turned to 180 degrees
- moved U6 8.56 mm to (97.0, 66.4)
- moved U2 8.21 mm to (90.5, 59.4)
- moved C6 8.10 mm to (106.5, 67.5)
- moved C9 7.48 mm to (125.5, 56.0)
- moved C3 7.02 mm to (97.0, 54.0)
- moved C4 7.02 mm to (97.0, 61.0)
- moved U1 7.02 mm to (111.5, 57.5)
- moved Y1 7.02 mm to (102.5, 59.9)
- moved Q1 5.59 mm to (124.0, 52.0)
- moved R11 4.53 mm to (90.5, 53.5)
- moved Q2 4.03 mm to (132.5, 49.0)
- moved C8 4.00 mm to (132.5, 42.5)
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Routing:
- net Net-(DS1-VDD): track 0.00 -> 253.4 mm, vias 0 -> 7
- net /btn_u: track 0.00 -> 104.1 mm, vias 0 -> 2
- net MOSI_ISP: track 0.00 -> 102.7 mm, vias 0 -> 2
- net /btn_ok: track 0.00 -> 95.2 mm, vias 0 -> 2
- net MISO_ISP: track 0.00 -> 90.2 mm, vias 0 -> 1
- net SCK_ISP: track 0.00 -> 77.8 mm, vias 0 -> 1
- net GND: track 13.6 -> 89.2 mm, vias 12 -> 35
- net RST_VCC: track 0.00 -> 66.9 mm, vias 0 -> 4
- net Net-(U1-PC2): track 0.00 -> 48.5 mm
- net RST_ISP: track 0.00 -> 40.8 mm, vias 0 -> 1
- net /R_SCL: track 0.00 -> 31.8 mm, vias 0 -> 4
- net /R_SDA: track 0.00 -> 31.7 mm, vias 0 -> 4
- net Net-(U3-DAC_L): track 0.00 -> 30.0 mm, vias 0 -> 1
- net Net-(U3-DAC_R): track 0.00 -> 29.9 mm
- net /A_TX: track 0.00 -> 24.0 mm, vias 0 -> 2
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Other:
- board size 114 x 39.5 mm -> 114 x 40 mm
