File: FMP3_PLAYER_CIRCUIT_ITER_2/FMP3_PLAYER.kicad_pcb (KiCad board)
At the start: 2 copper layers, 114 x 40 mm, 47 parts, among them J1 USB_C_Receptacle_PowerOnly_6P, J2 AudioJack3, J3 ISP, Q1 PMOS, Q2 PMOS, SW1 SW_L, SW2 SW_D, SW3 SW_R, SW4 SW_U, SW5 SW_SPDT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

Commit message: The DFPlayer NEEDS a fat decoupling cap...
Parts:
- added C12: 47u, Capacitor_THT:CP_Radial_D5.0mm_P2.50mm, F.Cu at (139.0, 50.0)
Routing:
- net Net-(Q1-S): track 7.90 -> 19.2 mm

Commit message: I swear to git this is the final pcb...
Parts:
- added C13: 100n, Capacitor_SMD:C_0805_2012Metric_Pad1.18x1.45mm_HandSolder, F.Cu at (159.0, 55.0)
- added C14: 100n, Capacitor_SMD:C_0805_2012Metric_Pad1.18x1.45mm_HandSolder, F.Cu at (153.0, 57.0)
Connections:
- J2 pad R: Net-(J2-PadR) -> Net-(C14-Pad1)
- J2 pad T: Net-(J2-PadT) -> Net-(C13-Pad1)
- U4 pad 10: Net-(J2-PadT) -> Net-(C13-Pad2)
- U4 pad 6: Net-(J2-PadR) -> Net-(C14-Pad2)
Routing:
- net Net-(J2-PadR): track 22.0 -> 0.00 mm, vias 2 -> 0
- net Net-(J2-PadT): track 15.1 -> 0.00 mm
- net Net-(C14-Pad1): track 0.00 -> 12.1 mm, vias 0 -> 2
- net Net-(C14-Pad2): track 0.00 -> 11.4 mm, vias 0 -> 2
- net Net-(C13-Pad2): track 0.00 -> 7.54 mm
- net Net-(C13-Pad1): track 0.00 -> 5.44 mm

Commit message: I realized after some prototyping my PMOS was bad, fixed now, i swear this better be the final...
Parts:
- removed Q1: PMOS, Package_TO_SOT_SMD:SOT-23_Handsoldering
- added Q3: BSS84, Package_TO_SOT_SMD:SOT-23_Handsoldering, F.Cu at (130.5, 46.0)
- added R14: 100k, Resistor_SMD:R_0805_2012Metric_Pad1.20x1.40mm_HandSolder, F.Cu at (127.0, 51.0)
- added R15: 100k, Resistor_SMD:R_0805_2012Metric_Pad1.20x1.40mm_HandSolder, F.Cu at (131.5, 49.0)
- Q2: value PMOS -> BSS84
- moved Q2 12.5 mm to (121.5, 55.0)
Connections:
- C12 pad 1: Net-(Q1-S) -> Net-(Q2-D)
- C8 pad 1: Net-(Q2-S) -> Net-(Q3-D)
- C9 pad 1: Net-(Q1-S) -> Net-(Q2-D)
- Q2 pad 1: Net-(DS1-VDD) -> Net-(Q2-G)
- Q2 pad 2: Net-(Q2-G) -> Net-(DS1-VDD)
- Q2 pad 3: Net-(Q2-S) -> Net-(Q2-D)
- U1 pad 23: Net-(Q1-G) -> Net-(Q2-G)
- U1 pad 24: Net-(Q2-G) -> Net-(Q3-G)
- U3 pad 1: Net-(Q1-S) -> Net-(Q2-D)
- U5 pad 5: Net-(Q2-S) -> Net-(Q3-D)
Routing:
- net Net-(Q3-G): track 0.00 -> 25.4 mm, vias 0 -> 4
- net Net-(Q1-S): track 19.2 -> 0.00 mm
- net Net-(Q2-D): track 0.00 -> 18.1 mm
- net Net-(Q2-S): track 10.2 -> 0.00 mm
- net Net-(Q3-D): track 0.00 -> 9.93 mm
- net Net-(DS1-VDD): track 253.4 -> 245.3 mm
- net Net-(Q1-G): track 7.89 -> 0.00 mm
- net GND: track 89.2 -> 95.4 mm, vias 35 -> 36
- net Net-(Q2-G): track 17.3 -> 19.4 mm
- net Net-(U1-PC2): track 48.5 -> 47.4 mm

Commit message: minor fix, used pulldowns instead of pullups by accident
Connections:
- C12 pad 1: Net-(Q2-D) -> Net-(DS1-VDD)
- C9 pad 1: Net-(Q2-D) -> Net-(DS1-VDD)
- Q2 pad 3: Net-(Q2-D) -> Net-(DS1-VDD)
- R14 pad 2: GND -> Net-(DS1-VDD)
- R15 pad 2: GND -> Net-(DS1-VDD)
- U3 pad 1: Net-(Q2-D) -> Net-(DS1-VDD)
Routing:
- net Net-(DS1-VDD): track 245.3 -> 276.3 mm
- net Net-(Q2-D): track 18.1 -> 0.00 mm
- net GND: track 95.4 -> 92.2 mm, vias 36 -> 34
Changed lines of the file:
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@@
 	(net 69 "Net-(C14-Pad2)")
 	(net 70 "Net-(Q3-D)")
-	(net 71 "Net-(Q2-D)")
-	(net 72 "Net-(Q3-G)")
+	(net 71 "Net-(Q3-G)")
 	(footprint "Resistor_SMD:R_0805_2012Metric_Pad1.20x1.40mm_HandSolder"
 		(layer "F.Cu")
@@
 			(layers "F.Cu" "F.Mask" "F.Paste")
 			(roundrect_rratio 0.208333)
-			(net 72 "Net-(Q3-G)")
+			(net 71 "Net-(Q3-G)")
 			(pintype "passive")
 		)
@@
 			(layers "F.Cu" "F.Mask" "F.Paste")
 			(roundrect_rratio 0.208333)
-			(net 1 "GND")
+			(net 6 "Net-(DS1-VDD)")
 			(pintype "passive")
 		)
@@
 			(layers "F.Cu" "F.Mask" "F.Paste")
 			(roundrect_rratio 0.25)
-			(net 72 "Net-(Q3-G)")
+			(net 71 "Net-(Q3-G)")
 			(pinfunction "PC1")
 			(pintype "bidirectional")
@@
 			(layers "*.Cu" "*.Mask")
 			(remove_unused_layers no)
-			(net 71 "Net-(Q2-D)")
+			(net 6 "Net-(DS1-VDD)")
 			(pinfunction "VCC")
 			(pintype "power_in")
@@
 			(layers "F.Cu" "F.Mask" "F.Paste")
 			(roundrect_rratio 0.25)
-			(net 71 "Net-(Q2-D)")
+			(net 6 "Net-(DS1-VDD)")
 			(pinfunction "D")
 			(pintype "passive")
@@
 			(layers "F.Cu" "F.Mask" "F.Paste")
 			(roundrect_rratio 0.25)
-			(net 72 "Net-(Q3-G)")
+			(net 71 "Net-(Q3-G)")
 			(pinfunction "G")
 			(pintype "input")
@@
 			(remove_unused_layers no)
 			(roundrect_rratio 0.15625)
-			(net 71 "Net-(Q2-D)")
+			(net 6 "Net-(DS1-VDD)")
 			(pintype "passive")
 		)
@@
 			(layers "F.Cu" "F.Mask" "F.Paste")
 			(roundrect_rratio 0.208333)
-			(net 1 "GND")
+			(net 6 "Net-(DS1-VDD)")
 			(pintype "passive")
 		)
@@
 			(layers "F.Cu" "F.Mask" "F.Paste")
 			(roundrect_rratio 0.212766)
-			(net 71 "Net-(Q2-D)")
+			(net 6 "Net-(DS1-VDD)")
 			(pintype "passive")
 		)
@@
 	)
 	(segment
-		(start 129 52)
-		(end 128 51)
-		(width 0.2)
-		(layer "F.Cu")
-		(net 1)
-	)
-	(segment
 		(start 109 43.5)
 		(end 110.5 45)
@@
 	)
 	(segment
-		(start 133.5 49)
-		(end 134 48.5)
-		(width 0.2)
-		(layer "F.Cu")
-		(net 1)
-	)
-	(segment
 		(start 127.1 40)
 		(end 127.1 42.829655)
@@
 	)
 	(segment
-		(start 132.5 49)
-		(end 133.5 49)
-		(width 0.2)
-		(layer "F.Cu")
-		(net 1)
-	)
-	(segment
 		(start 111.5 48.5)
 		(end 110.5 47.5)
@@
 	)
 	(via
-		(at 129 52)
-		(size 0.6)
-		(drill 0.3)
-		(layers "F.Cu" "B.Cu")
-		(net 1)
-	)
-	(via
-		(at 134 48.5)
-		(size 0.6)
-		(drill 0.3)
-		(layers "F.Cu" "B.Cu")
-		(net 1)
-	)
-	(via
 		(at 90.5 59.5)
 		(size 0.6)
@@
 	)
 	(segment
+		(start 139 50)
+		(end 138 49)
+		(width 0.2)
+		(layer "F.Cu")
+		(net 6)
+	)
+	(segment
 		(start 91.04 39.5)
 		(end 92.191 38.349)
@@
 	)
 	(segment
+		(start 138 49)
+		(end 132.5 49)
+		(width 0.2)
+		(layer "F.Cu")
+		(net 6)
+	)
+	(segment
 		(start 96 67.854468)
 		(end 96 67.5)
@@
 	)
 	(segment
+		(start 123 55)
+		(end 125.4625 55)
+		(width 0.2)
+		(layer "F.Cu")
+		(net 6)
+	)
+	(segment
 		(start 168 47.05)
 		(end 172.05 43)
@@
 	)
 	(segment
+		(start 143 47.5)
+		(end 131 47.5)
+		(width 0.2)
+		(layer "F.Cu")
+		(net 6)
+	)
+	(segment
 		(start 182.5 53.5)
 		(end 180.95 53.5)
@@
 	)
 	(segment
+		(start 125.4625 55)
+		(end 125.5 54.9625)
+		(width 0.2)
+		(layer "F.Cu")
+		(net 6)
+	)
+	(segment
 		(start 120.4 52.448)
 		(end 121.251 53.299)
@@
 	)
 	(segment
+		(start 132.5 49)
+		(end 131 47.5)
+		(width 0.2)
+		(layer "F.Cu")
+		(net 6)
+	)
+	(segment
 		(start 185.68516 46.099)
 		(end 186.001 46.41484)
@@
 	)
 	(segment
+		(start 129 54.34)
+		(end 128.3775 54.9625)
+		(width 0.2)
+		(layer "F.Cu")
+		(net 6)
+	)
+	(segment
 		(start 172.05 68)
 		(end 180.95 68)
@@
 	)
 	(segment
-		(start 143 47.5)
+		(start 131 47.5)
 		(end 129.55 47.5)
 		(width 0.2)
@@
 	)
 	(segment
+		(start 128.3775 54.9625)
+		(end 125.5 54.9625)
+		(width 0.2)
+		(layer "F.Cu")
+		(net 6)
+	)
+	(segment
+		(start 128 51)
+		(end 128 52.874)
+		(width 0.2)
+		(layer "F.Cu")
+		(net 6)
+	)
+	(segment
 		(start 180.95 53.5)
 		(end 172.05 53.5)
@@
 	)
 	(segment
+		(start 129.466 54.34)
+		(end 129 54.34)
+		(width 0.2)
+		(layer "F.Cu")
+		(net 6)
+	)
+	(segment
+		(start 128 52.874)
+		(end 129.466 54.34)
+		(width 0.2)
+		(layer "F.Cu")
+		(net 6)
+	)
+	(segment
 		(start 120 48)
 		(end 120 46.5)
@@
 	)
 	(segment
+		(start 133.806 50)
+		(end 129.466 54.34)
+		(width 0.2)
+		(layer "B.Cu")
+		(net 6)
+	)
+	(segment
 		(start 156.1 46)
 		(end 153 46)
@@
 	)
 	(segment
+		(start 139 50)
+		(end 133.806 50)
+		(width 0.2)
+		(layer "B.Cu")
+		(net 6)
+	)
+	(segment
 		(start 120.4 52.448)
 		(end 120 52.048)
@@
 	)
 	(segment
-		(start 123 55)
-		(end 125.4625 55)
-		(width 0.2)
-		(layer "F.Cu")
-		(net 71)
-	)
-	(segment
-		(start 125.4625 55)
-		(end 125.5 54.9625)
-		(width 0.2)
-		(layer "F.Cu")
-		(net 71)
-	)
-	(segment
-		(start 129 54.34)
-		(end 128.3775 54.9625)
-		(width 0.2)
-		(layer "F.Cu")
-		(net 71)
-	)
-	(segment
-		(start 128.3775 54.9625)
-		(end 125.5 54.9625)
-		(width 0.2)
-		(layer "F.Cu")
-		(net 71)
-	)
-	(segment
-		(start 129.466 54.34)
-		(end 129 54.34)
-		(width 0.2)
-		(layer "F.Cu")
-		(net 71)
-	)
-	(segment
-		(start 133.806 50)
-		(end 129.466 54.34)
-		(width 0.2)
-		(layer "B.Cu")
-		(net 71)
-	)
-	(segment
-		(start 139 50)
-		(end 133.806 50)
-		(width 0.2)
-		(layer "B.Cu")
-		(net 71)
-	)
-	(segment
 		(start 128.95 45)
 		(end 127.65326 45)
 		(width 0.2)
 		(layer "F.Cu")
-		(net 72)
+		(net 71)
 	)
 	(segment
@@
 		(width 0.2)
 		(layer "F.Cu")
-		(net 72)
+		(net 71)
 	)
 	(segment
@@
 		(width 0.2)
 		(layer "F.Cu")
-		(net 72)
+		(net 71)
 	)
 	(segment
@@
 		(width 0.2)
 		(layer "F.Cu")
-		(net 72)
+		(net 71)
 	)
 	(segment
@@
 		(width 0.2)
 		(layer "F.Cu")
-		(net 72)
+		(net 71)
 	)
 	(segment
@@
 		(width 0.2)
 		(layer "F.Cu")
-		(net 72)
+		(net 71)
 	)
 	(segment
@@
 		(width 0.2)
 		(layer "F.Cu")
-		(net 72)
+		(net 71)
 	)
 	(segment
@@
 		(width 0.2)
 		(layer "F.Cu")
-		(net 72)
+		(net 71)
 	)
 	(segment
@@
 		(width 0.2)
 		(layer "F.Cu")
-		(net 72)
+		(net 71)
 	)
 	(segment
@@
 		(width 0.2)
 		(layer "F.Cu")
-		(net 72)
+		(net 71)
 	)
 	(segment
@@
 		(width 0.2)
 		(layer "F.Cu")
-		(net 72)
+		(net 71)
 	)
 	(segment
@@
 		(width 0.2)
 		(layer "F.Cu")
-		(net 72)
+		(net 71)
 	)
 	(via
@@
 		(drill 0.3)
 		(layers "F.Cu" "B.Cu")
-		(net 72)
+		(net 71)
 	)
 	(via
@@
 		(drill 0.3)
 		(layers "F.Cu" "B.Cu")
-		(net 72)
+		(net 71)
 	)
 	(via
@@
 		(drill 0.3)
 		(layers "F.Cu" "B.Cu")
-		(net 72)
+		(net 71)
 	)
 	(via
@@
 		(drill 0.3)
 		(layers "F.Cu" "B.Cu")
-		(net 72)
+		(net 71)
 	)
 	(segment
@@
 		(width 0.2)
 		(layer "B.Cu")
-		(net 72)
+		(net 71)
 	)
 	(segment
@@
 		(width 0.2)
 		(layer "B.Cu")
-		(net 72)
+		(net 71)
 	)
 	(segment
@@
 		(width 0.2)
 		(layer "B.Cu")
-		(net 72)
+		(net 71)
 	)
 	(segment
@@
 		(width 0.2)
 		(layer "B.Cu")
-		(net 72)
+		(net 71)
 	)
 	(segment
@@
 		(width 0.2)
 		(layer "B.Cu")
-		(net 72)
+		(net 71)
 	)
 	(zone

Commit message: another minor fix, i should really go sleep...
Connections:
- C12 pad 1: Net-(DS1-VDD) -> Net-(Q2-D)
- C9 pad 1: Net-(DS1-VDD) -> Net-(Q2-D)
- Q2 pad 3: Net-(DS1-VDD) -> Net-(Q2-D)
- U3 pad 1: Net-(DS1-VDD) -> Net-(Q2-D)
Routing:
- net Net-(DS1-VDD): track 276.3 -> 253.3 mm, vias 7 -> 9
- net Net-(Q2-D): track 0.00 -> 18.1 mm
Changed lines of the file:
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@@
 	(net 70 "Net-(Q3-D)")
 	(net 71 "Net-(Q3-G)")
+	(net 72 "Net-(Q2-D)")
 	(footprint "Resistor_SMD:R_0805_2012Metric_Pad1.20x1.40mm_HandSolder"
 		(layer "F.Cu")
@@
 			(layers "*.Cu" "*.Mask")
 			(remove_unused_layers no)
-			(net 6 "Net-(DS1-VDD)")
+			(net 72 "Net-(Q2-D)")
 			(pinfunction "VCC")
 			(pintype "power_in")
@@
 			(layers "F.Cu" "F.Mask" "F.Paste")
 			(roundrect_rratio 0.25)
-			(net 6 "Net-(DS1-VDD)")
+			(net 72 "Net-(Q2-D)")
 			(pinfunction "D")
 			(pintype "passive")
@@
 			(remove_unused_layers no)
 			(roundrect_rratio 0.15625)
-			(net 6 "Net-(DS1-VDD)")
+			(net 72 "Net-(Q2-D)")
 			(pintype "passive")
 		)
@@
 			(layers "F.Cu" "F.Mask" "F.Paste")
 			(roundrect_rratio 0.212766)
-			(net 6 "Net-(DS1-VDD)")
+			(net 72 "Net-(Q2-D)")
 			(pintype "passive")
 		)
@@
 	)
 	(segment
+		(start 128.5 48)
+		(end 128.5 47.45)
+		(width 0.2)
+		(layer "F.Cu")
+		(net 6)
+	)
+	(segment
 		(start 184.049 46.099)
 		(end 185.68516 46.099)
@@
 	)
 	(segment
+		(start 128 51)
+		(end 129.1 51)
+		(width 0.2)
+		(layer "F.Cu")
+		(net 6)
+	)
+	(segment
 		(start 91.04 39.5)
 		(end 95.399 43.859)
@@
 	)
 	(segment
-		(start 139 50)
-		(end 138 49)
-		(width 0.2)
-		(layer "F.Cu")
-		(net 6)
-	)
-	(segment
 		(start 91.04 39.5)
 		(end 92.191 38.349)
@@
 	)
 	(segment
-		(start 138 49)
-		(end 132.5 49)
-		(width 0.2)
-		(layer "F.Cu")
-		(net 6)
-	)
-	(segment
 		(start 96 67.854468)
 		(end 96 67.5)
@@
 	)
 	(segment
-		(start 123 55)
-		(end 125.4625 55)
-		(width 0.2)
-		(layer "F.Cu")
-		(net 6)
-	)
-	(segment
 		(start 168 47.05)
 		(end 172.05 43)
@@
 	)
 	(segment
-		(start 125.4625 55)
-		(end 125.5 54.9625)
-		(width 0.2)
-		(layer "F.Cu")
-		(net 6)
-	)
-	(segment
 		(start 120.4 52.448)
 		(end 121.251 53.299)
@@
 	)
 	(segment
-		(start 129 54.34)
-		(end 128.3775 54.9625)
-		(width 0.2)
-		(layer "F.Cu")
-		(net 6)
-	)
-	(segment
 		(start 172.05 68)
 		(end 180.95 68)
@@
 	)
 	(segment
-		(start 128.3775 54.9625)
-		(end 125.5 54.9625)
+		(start 129.1 51)
+		(end 129.5 50.6)
 		(width 0.2)
 		(layer "F.Cu")
@@
 	)
 	(segment
-		(start 128 51)
-		(end 128 52.874)
+		(start 128.5 47.45)
+		(end 129 46.95)
 		(width 0.2)
 		(layer "F.Cu")
@@
 	)
 	(segment
-		(start 129.466 54.34)
-		(end 129 54.34)
-		(width 0.2)
-		(layer "F.Cu")
-		(net 6)
-	)
-	(segment
-		(start 128 52.874)
-		(end 129.466 54.34)
-		(width 0.2)
-		(layer "F.Cu")
-		(net 6)
-	)
-	(segment
 		(start 120 48)
 		(end 120 46.5)
@@
 	)
 	(via
+		(at 129.5 50.6)
+		(size 0.6)
+		(drill 0.3)
+		(layers "F.Cu" "B.Cu")
+		(net 6)
+	)
+	(via
 		(at 168 62.5)
 		(size 0.6)
@@
 	)
 	(via
+		(at 128.5 48)
+		(size 0.6)
+		(drill 0.3)
+		(layers "F.Cu" "B.Cu")
+		(net 6)
+	)
+	(via
 		(at 120.4 52.448)
 		(size 0.6)
@@
 	)
 	(segment
-		(start 133.806 50)
-		(end 129.466 54.34)
+		(start 129.5 49)
+		(end 128.5 48)
 		(width 0.2)
 		(layer "B.Cu")
@@
 	)
 	(segment
-		(start 139 50)
-		(end 133.806 50)
+		(start 120.4 52.448)
+		(end 120 52.048)
 		(width 0.2)
 		(layer "B.Cu")
@@
 	)
 	(segment
-		(start 120.4 52.448)
-		(end 120 52.048)
+		(start 129.5 50.6)
+		(end 129.5 49)
 		(width 0.2)
 		(layer "B.Cu")
@@
 		(net 71)
 	)
+	(segment
+		(start 123 55)
+		(end 125.4625 55)
+		(width 0.2)
+		(layer "F.Cu")
+		(net 72)
+	)
+	(segment
+		(start 125.4625 55)
+		(end 125.5 54.9625)
+		(width 0.2)
+		(layer "F.Cu")
+		(net 72)
+	)
+	(segment
+		(start 129 54.34)
+		(end 128.3775 54.9625)
+		(width 0.2)
+		(layer "F.Cu")
+		(net 72)
+	)
+	(segment
+		(start 128.3775 54.9625)
+		(end 125.5 54.9625)
+		(width 0.2)
+		(layer "F.Cu")
+		(net 72)
+	)
+	(segment
+		(start 129.466 54.34)
+		(end 129 54.34)
+		(width 0.2)
+		(layer "F.Cu")
+		(net 72)
+	)
+	(segment
+		(start 133.806 50)
+		(end 129.466 54.34)
+		(width 0.2)
+		(layer "B.Cu")
+		(net 72)
+	)
+	(segment
+		(start 139 50)
+		(end 133.806 50)
+		(width 0.2)
+		(layer "B.Cu")
+		(net 72)
+	)
 	(zone
